File: ZXClone/zxclone.brd (EAGLE design)
At the start: 38.1 x 38.1 mm, 18 parts, among them IC1 TLC272P

Commit message: Ready to send gerber files
Routing:
- net GND: track 0.00 -> 67.9 mm
- net N$1: track 0.00 -> 55.1 mm
- net N$5: track 0.00 -> 36.3 mm
- net SIG: track 0.00 -> 34.5 mm
- net N$2: track 0.00 -> 29.2 mm
- net N$7: track 0.00 -> 25.2 mm
- net N$3: track 0.00 -> 19.2 mm
- net N$4: track 0.00 -> 18.6 mm
- net VCC: track 0.00 -> 10.3 mm
Other:
- board text added: "0.1uF"
- board text added: "100k"
- board text added: "12R"
- board text added: "1k"
- board text added: "22k"
- board text added: "22uF"
- board text added: "470uF"
- board text added: "68k"
- board text added: "TLC272P"
