File: AnalogIntensityBar/AnalogIntensityBar.brd (EAGLE design)
At the start: 30.5 x 27.9 mm, 34 parts, among them Q1 20Mhz

Commit message: Cleanup
Parts:
- moved BAR1 1.52 mm to (27.8, 22.0)
- moved RBAR1 1.52 mm to (24.8, 22.0)
- moved BAR2 1.27 mm to (27.8, 20.3)
- moved RBAR2 1.27 mm to (24.8, 20.3)
- moved BAR3 1.02 mm to (27.8, 18.7)
- moved RBAR3 1.02 mm to (24.8, 18.7)
- moved BAR4 0.76 mm to (27.8, 17.0)
- moved RBAR4 0.76 mm to (24.8, 17.0)
- moved BAR10 0.76 mm to (27.8, 7.11)
- moved RBAR10 0.76 mm to (24.8, 7.11)
- moved BAR5 0.51 mm to (27.8, 15.4)
- moved BAR9 0.51 mm to (27.8, 8.76)
- moved RBAR5 0.51 mm to (24.8, 15.4)
- moved RBAR9 0.51 mm to (24.8, 8.76)
- moved BAR6 0.25 mm to (27.8, 13.7)
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Routing:
- net GND: track 112.3 -> 124.4 mm, vias 2 -> 3
- net MISO: track 31.3 -> 37.9 mm, vias 2 -> 1
- net MOSI: track 47.0 -> 42.5 mm
- net N$1: track 4.29 -> 5.59 mm
- net N$2: track 4.24 -> 5.11 mm
- net N$5: track 4.19 -> 4.98 mm
Other:
- board text added: "ISP"
