File: ZXCloneSMD/zxclone.sch (EAGLE design)
At the start: 18 parts, among them IC1 TLC272D

Commit message: On the way to a second proto board
Parts:
- added R8: TRIMPOT-2, SparkFun-Electromechanical:TRIMPOT-2
- C1: device resistor:CPOL-USE2.5-7 -> rcl:CPOL-USCT7343
- R1, R2, R3, R4, R5, R6: device resistor:R-US_R0805 -> resistor:R-US_R0402
Connections:
- new net N$6: R5.2, R8.CCW
- net GND: now also U$1.2; no longer U$1.1
- net N$1: now also R8.WIPER; no longer R5.2
- net N$7: now also U$1.1; no longer U$1.2
Other:
- moved on the sheet: U$1
Changed lines of the file:
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@@
 <class number="0" name="default" width="0" drill="0">
+</class>
+<class number="1" name="ground" width="0.4064" drill="0">
+</class>
+<class number="2" name="vcc" width="0.4064" drill="0">
 </class>
 </classes>
 <parts>
 <part name="IC1" library="linear" deviceset="TLC272" device="D" value="TLC272D"/>
-<part name="R1" library="resistor" deviceset="R-US_" device="R0805" value="22k"/>
-<part name="R2" library="resistor" deviceset="R-US_" device="R0805" value="100k"/>
-<part name="R3" library="resistor" deviceset="R-US_" device="R0805" value="1k"/>
-<part name="R4" library="resistor" deviceset="R-US_" device="R0805" value="100k"/>
-<part name="R5" library="resistor" deviceset="R-US_" device="R0805" value="68k"/>
-<part name="R6" library="resistor" deviceset="R-US_" device="R0805" value="1k"/>
+<part name="R1" library="resistor" deviceset="R-US_" device="R0402" value="22k"/>
+<part name="R2" library="resistor" deviceset="R-US_" device="R0402" value="100k"/>
+<part name="R3" library="resistor" deviceset="R-US_" device="R0402" value="1k"/>
+<part name="R4" library="resistor" deviceset="R-US_" device="R0402" value="100k"/>
+<part name="R5" library="resistor" deviceset="R-US_" device="R0402" value="68k"/>
+<part name="R6" library="resistor" deviceset="R-US_" device="R0402" value="1k"/>
 <part name="R7" library="resistor" deviceset="R-US_" device="R0805" value="12R"/>
-<part name="C1" library="resistor" deviceset="CPOL-US" device="E2.5-7" value="470uF"/>
+<part name="C1" library="rcl" deviceset="CPOL-US" device="CT7343" value="470uF"/>
 <part name="U$1" library="SparkFun-Sensors" deviceset="MIC" device="9.7MM"/>
 <part name="FRAME1" library="SparkFun-Aesthetics" deviceset="FRAME-LETTER" device=""/>
@@
 <part name="SUPPLY2" library="SparkFun-Aesthetics" deviceset="VCC" device=""/>
 <part name="GND2" library="SparkFun-Aesthetics" deviceset="GND" device=""/>
+<part name="R8" library="SparkFun-Electromechanical" deviceset="TRIMPOT" device="-2"/>
 </parts>
 <sheets>
@@
 <instance part="R7" gate="G$1" x="147.32" y="152.4"/>
 <instance part="C1" gate="G$1" x="101.6" y="144.78"/>
-<instance part="U$1" gate="G$1" x="55.88" y="116.84" rot="R90"/>
+<instance part="U$1" gate="G$1" x="53.34" y="119.38" rot="MR270"/>
 <instance part="FRAME1" gate="G$1" x="-2.54" y="7.62"/>
 <instance part="FRAME1" gate="G$2" x="144.78" y="7.62"/>
@@
 <instance part="SUPPLY2" gate="1" x="139.7" y="129.54"/>
 <instance part="GND2" gate="1" x="139.7" y="111.76"/>
+<instance part="R8" gate="R?" x="139.7" y="142.24"/>
 </instances>
 <busses>
@@
 </segment>
 </net>
-<net name="GND" class="0">
+<net name="GND" class="1">
 <segment>
 <pinref part="R6" gate="G$1" pin="1"/>
@@
 </segment>
 <segment>
-<pinref part="U$1" gate="G$1" pin="1"/>
-<wire x1="58.42" y1="116.84" x2="60.96" y2="116.84" width="0.1524" layer="91"/>
 <wire x1="60.96" y1="116.84" x2="60.96" y2="106.68" width="0.1524" layer="91"/>
 <pinref part="R3" gate="G$1" pin="2"/>
@@
 <junction x="60.96" y="96.52"/>
 <pinref part="GND4" gate="1" pin="GND"/>
+<pinref part="U$1" gate="G$1" pin="2"/>
+<wire x1="60.96" y1="116.84" x2="55.88" y2="116.84" width="0.1524" layer="91"/>
 </segment>
 <segment>
@@
 </segment>
 </net>
-<net name="VCC" class="0">
+<net name="VCC" class="2">
 <segment>
 <pinref part="SUPPLY1" gate="1" pin="VCC"/>
@@
 </segment>
 </net>
-<net name="N$1" class="0">
+<net name="N$1" class="2">
 <segment>
 <pinref part="R7" gate="G$1" pin="1"/>
-<wire x1="142.24" y1="152.4" x2="127" y2="152.4" width="0.1524" layer="91"/>
-<pinref part="R5" gate="G$1" pin="2"/>
-<wire x1="127" y1="152.4" x2="127" y2="147.32" width="0.1524" layer="91"/>
-<wire x1="127" y1="152.4" x2="101.6" y2="152.4" width="0.1524" layer="91"/>
-<junction x="127" y="152.4"/>
+<wire x1="142.24" y1="152.4" x2="139.7" y2="152.4" width="0.1524" layer="91"/>
 <pinref part="C1" gate="G$1" pin="+"/>
+<wire x1="134.62" y1="152.4" x2="101.6" y2="152.4" width="0.1524" layer="91"/>
 <wire x1="101.6" y1="152.4" x2="101.6" y2="147.32" width="0.1524" layer="91"/>
 <pinref part="R1" gate="G$1" pin="1"/>
 <wire x1="101.6" y1="152.4" x2="91.44" y2="152.4" width="0.1524" layer="91"/>
 <junction x="101.6" y="152.4"/>
+<pinref part="R8" gate="R?" pin="WIPER"/>
+<wire x1="134.62" y1="152.4" x2="139.7" y2="152.4" width="0.1524" layer="91"/>
+<wire x1="139.7" y1="152.4" x2="139.7" y2="147.32" width="0.1524" layer="91"/>
 </segment>
 </net>
@@
 </segment>
 </net>
-<net name="N$7" class="0">
+<net name="N$7" class="2">
 <segment>
 <pinref part="R1" gate="G$1" pin="2"/>
 <wire x1="81.28" y1="152.4" x2="60.96" y2="152.4" width="0.1524" layer="91"/>
 <wire x1="60.96" y1="152.4" x2="60.96" y2="119.38" width="0.1524" layer="91"/>
-<pinref part="U$1" gate="G$1" pin="2"/>
-<wire x1="60.96" y1="119.38" x2="58.42" y2="119.38" width="0.1524" layer="91"/>
 <wire x1="60.96" y1="119.38" x2="68.58" y2="119.38" width="0.1524" layer="91"/>
+<pinref part="C3" gate="G$1" pin="1"/>
+<pinref part="U$1" gate="G$1" pin="1"/>
+<wire x1="60.96" y1="119.38" x2="55.88" y2="119.38" width="0.1524" layer="91"/>
 <junction x="60.96" y="119.38"/>
-<pinref part="C3" gate="G$1" pin="1"/>
-</segment>
-</net>
+</segment>
+</net>
+<net name="N$6" class="0">
+<segment>
+<pinref part="R8" gate="R?" pin="CCW"/>
+<wire x1="134.62" y1="142.24" x2="134.62" y2="147.32" width="0.1524" layer="91"/>
+<pinref part="R5" gate="G$1" pin="2"/>
+<wire x1="134.62" y1="147.32" x2="127" y2="147.32" width="0.1524" layer="91"/>
+</segment>
+</net>

Commit message: Working revision with LED and trimpot
Parts:
- added LED1: (no value), led:LEDSML0603
- added R9: 1k, resistor:R-US_R0402
- C1: device rcl:CPOL-USCT7343 -> resistor:CPOL-USE2.5-7
- R5: value 68k -> 30k
- R8: value TRIMPOT-2 -> TRIMPOT 25K
Connections:
- new net N$8: LED1.A, R9.1
- net GND: now also LED1.C
- net N$6: now also R8.CW; no longer R8.CCW
- net SIG: now also R9.2
Other:
- moved on the sheet: R7, R8
Changed lines of the file:
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@@
 <part name="R3" library="resistor" deviceset="R-US_" device="R0402" value="1k"/>
 <part name="R4" library="resistor" deviceset="R-US_" device="R0402" value="100k"/>
-<part name="R5" library="resistor" deviceset="R-US_" device="R0402" value="68k"/>
+<part name="R5" library="resistor" deviceset="R-US_" device="R0402" value="30k"/>
 <part name="R6" library="resistor" deviceset="R-US_" device="R0402" value="1k"/>
 <part name="R7" library="resistor" deviceset="R-US_" device="R0805" value="12R"/>
-<part name="C1" library="rcl" deviceset="CPOL-US" device="CT7343" value="470uF"/>
+<part name="C1" library="resistor" deviceset="CPOL-US" device="E2.5-7" value="470uF"/>
 <part name="U$1" library="SparkFun-Sensors" deviceset="MIC" device="9.7MM"/>
 <part name="FRAME1" library="SparkFun-Aesthetics" deviceset="FRAME-LETTER" device=""/>
@@
 <part name="SUPPLY2" library="SparkFun-Aesthetics" deviceset="VCC" device=""/>
 <part name="GND2" library="SparkFun-Aesthetics" deviceset="GND" device=""/>
-<part name="R8" library="SparkFun-Electromechanical" deviceset="TRIMPOT" device="-2"/>
+<part name="R8" library="SparkFun-Electromechanical" deviceset="TRIMPOT" device="-2" value="TRIMPOT 25K"/>
+<part name="R9" library="resistor" deviceset="R-US_" device="R0402" value="1k"/>
+<part name="LED1" library="led" deviceset="LED" device="SML0603"/>
+<part name="GND5" library="SparkFun-Aesthetics" deviceset="GND" device=""/>
 </parts>
 <sheets>
@@
 <instance part="R5" gate="G$1" x="127" y="142.24" rot="R90"/>
 <instance part="R6" gate="G$1" x="111.76" y="134.62"/>
-<instance part="R7" gate="G$1" x="147.32" y="152.4"/>
+<instance part="R7" gate="G$1" x="154.94" y="152.4"/>
 <instance part="C1" gate="G$1" x="101.6" y="144.78"/>
 <instance part="U$1" gate="G$1" x="53.34" y="119.38" rot="MR270"/>
@@
 <instance part="SUPPLY2" gate="1" x="139.7" y="129.54"/>
 <instance part="GND2" gate="1" x="139.7" y="111.76"/>
-<instance part="R8" gate="R?" x="139.7" y="142.24"/>
+<instance part="R8" gate="R?" x="144.78" y="142.24" rot="MR0"/>
+<instance part="R9" gate="G$1" x="170.18" y="111.76" rot="R90"/>
+<instance part="LED1" gate="G$1" x="170.18" y="101.6"/>
+<instance part="GND5" gate="1" x="170.18" y="91.44"/>
 </instances>
 <busses>
@@
 <pinref part="GND2" gate="1" pin="GND"/>
 </segment>
+<segment>
+<pinref part="LED1" gate="G$1" pin="C"/>
+<pinref part="GND5" gate="1" pin="GND"/>
+<wire x1="170.18" y1="96.52" x2="170.18" y2="93.98" width="0.1524" layer="91"/>
+</segment>
 </net>
 <net name="VCC" class="2">
@@
 <wire x1="165.1" y1="157.48" x2="165.1" y2="152.4" width="0.1524" layer="91"/>
 <pinref part="R7" gate="G$1" pin="2"/>
-<wire x1="165.1" y1="152.4" x2="152.4" y2="152.4" width="0.1524" layer="91"/>
+<wire x1="165.1" y1="152.4" x2="160.02" y2="152.4" width="0.1524" layer="91"/>
 </segment>
 <segment>
@@
 <segment>
 <pinref part="R7" gate="G$1" pin="1"/>
-<wire x1="142.24" y1="152.4" x2="139.7" y2="152.4" width="0.1524" layer="91"/>
+<wire x1="149.86" y1="152.4" x2="144.78" y2="152.4" width="0.1524" layer="91"/>
 <pinref part="C1" gate="G$1" pin="+"/>
-<wire x1="134.62" y1="152.4" x2="101.6" y2="152.4" width="0.1524" layer="91"/>
+<wire x1="144.78" y1="152.4" x2="101.6" y2="152.4" width="0.1524" layer="91"/>
 <wire x1="101.6" y1="152.4" x2="101.6" y2="147.32" width="0.1524" layer="91"/>
 <pinref part="R1" gate="G$1" pin="1"/>
@@
 <junction x="101.6" y="152.4"/>
 <pinref part="R8" gate="R?" pin="WIPER"/>
-<wire x1="134.62" y1="152.4" x2="139.7" y2="152.4" width="0.1524" layer="91"/>
-<wire x1="139.7" y1="152.4" x2="139.7" y2="147.32" width="0.1524" layer="91"/>
+<wire x1="144.78" y1="152.4" x2="144.78" y2="147.32" width="0.1524" layer="91"/>
 </segment>
 </net>
@@
 <wire x1="147.32" y1="121.92" x2="157.48" y2="121.92" width="0.1524" layer="91"/>
 <label x="177.8" y="121.92" size="1.778" layer="95"/>
-<wire x1="157.48" y1="121.92" x2="177.8" y2="121.92" width="0.1524" layer="91"/>
+<wire x1="157.48" y1="121.92" x2="170.18" y2="121.92" width="0.1524" layer="91"/>
+<wire x1="170.18" y1="121.92" x2="177.8" y2="121.92" width="0.1524" layer="91"/>
 <wire x1="157.48" y1="121.92" x2="157.48" y2="106.68" width="0.1524" layer="91"/>
 <junction x="157.48" y="121.92"/>
 <pinref part="C2" gate="G$1" pin="1"/>
+<pinref part="R9" gate="G$1" pin="2"/>
+<wire x1="170.18" y1="121.92" x2="170.18" y2="116.84" width="0.1524" layer="91"/>
+<junction x="170.18" y="121.92"/>
 </segment>
 <segment>
@@
 <net name="N$6" class="0">
 <segment>
-<pinref part="R8" gate="R?" pin="CCW"/>
-<wire x1="134.62" y1="142.24" x2="134.62" y2="147.32" width="0.1524" layer="91"/>
 <pinref part="R5" gate="G$1" pin="2"/>
-<wire x1="134.62" y1="147.32" x2="127" y2="147.32" width="0.1524" layer="91"/>
-</segment>
-</net>
+<wire x1="139.7" y1="147.32" x2="127" y2="147.32" width="0.1524" layer="91"/>
+<pinref part="R8" gate="R?" pin="CW"/>
+<wire x1="139.7" y1="142.24" x2="139.7" y2="147.32" width="0.1524" layer="91"/>
+</segment>
+</net>
+<net name="N$8" class="0">
+<segment>
+<pinref part="R9" gate="G$1" pin="1"/>
+<pinref part="LED1" gate="G$1" pin="A"/>
+<wire x1="170.18" y1="106.68" x2="170.18" y2="104.14" width="0.1524" layer="91"/>
+</segment>
+</net>
